File: KiCad/9.0/projects/Soul_PS_Dash_V1/Soul_PS_Dash_V1.kicad_sch (KiCad schematic)
At the start: 30 parts, among them J1 +12V-GND, J10 GND-Fuel, J2 IGN-LSG-RSG-LS1-LS2, J3 C-CAN, J4 C-CAN, J5 C-CAN SPI, J6 B-CAN, J7 B-CAN, J8 B-CAN SPI, J9 Jumper Holder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

Commit message: KiCad: update Soul_PS_Dash_V1
Parts:
- removed BZ1: Buzzer, Buzzer_Beeper:Buzzer_12x9.5RM7.6, symbol Device:Buzzer
- removed J6: B-CAN, Connector_PinSocket_2.54mm:PinSocket_1x02_P2.54mm_Vertical, symbol Connector:Conn_01x02_Pin
- removed J7: B-CAN, Connector_JST:JST_XH_B2B-XH-A_1x02_P2.50mm_Vertical, symbol Connector:Conn_01x02_Pin
- removed J8: B-CAN SPI, Connector_PinSocket_2.54mm:PinSocket_1x07_P2.54mm_Vertical, symbol Connector:Conn_01x07_Pin
- removed J9: Jumper Holder, Connector_PinHeader_2.54mm:PinHeader_1x02_P2.54mm_Vertical, symbol Connector:Conn_01x02_Pin
- J2: value IGN-LSG-RSG-LS1-LS2 -> IGN-ILL-SRS-OIL-ALT_L
- U1, U2: footprint Package_DIP:DIP-18_W7.62mm_Socket -> Package_DIP:DIP-18_W7.62mm
- U3: footprint Package_DIP:DIP-16_W7.62mm_Socket -> Package_DIP:DIP-16_W7.62mm
- renumbered J10 to J6
Connections:
- net CAN_CS_B: no longer names the net of A1.10 (D7)
- no-connect marks 20 -> 22
Other:
- note removed: "LS: Low-Side Switch"
