File: KiCad/9.0/projects/Soul_PS_Dash_V1/Soul_PS_Dash_V1.kicad_pcb (KiCad board)
At the start: 2 copper layers, 109 x 64 mm, 30 parts, among them J1 +12V-GND, J10 GND-Fuel, J2 IGN-LSG-RSG-LS1-LS2, J3 C-CAN, J4 C-CAN, J5 C-CAN SPI, J6 B-CAN, J7 B-CAN, J8 B-CAN SPI, J9 Jumper Holder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

Commit message: KiCad: update Soul_PS_Dash_V1
Parts:
- removed BZ1: Buzzer, Buzzer_Beeper:Buzzer_12x9.5RM7.6
- removed the J6 at (193.4, 98.7)
- removed J7: B-CAN, Connector_JST:JST_XH_B2B-XH-A_1x02_P2.50mm_Vertical
- removed J8: B-CAN SPI, Connector_PinSocket_2.54mm:PinSocket_1x07_P2.54mm_Vertical
- removed J9: Jumper Holder, Connector_PinHeader_2.54mm:PinHeader_1x02_P2.54mm_Vertical
- J2: value IGN-LSG-RSG-LS1-LS2 -> IGN-ILL-SRS-OIL-ALT_L
- U1, U2: footprint Package_DIP:DIP-18_W7.62mm_Socket -> Package_DIP:DIP-18_W7.62mm
- U3: footprint Package_DIP:DIP-16_W7.62mm_Socket -> Package_DIP:DIP-16_W7.62mm
- moved Q2 5.00 mm to (150.0, 55.4)
- moved Q3 5.00 mm to (155.7, 55.4)
- moved R2 5.00 mm to (151.2, 59.5)
- moved R3 5.00 mm to (157.0, 59.5)
- moved C1 3.41 mm to (195.0, 82.0)
- moved J6 0.50 mm to (188.0, 55.0)
- renumbered J10 to J6
Connections:
- A1 pad 10: /CAN_CS_B -> unconnected-(A1-D7-Pad10)
- A1 pad 12: Net-(A1-D9) -> unconnected-(A1-D9-Pad12)
Routing:
- net Net-(A1-D9): track 112.4 -> 0.00 mm
- net /B-CAN_P: track 81.5 -> 0.00 mm, vias 1 -> 0
- net /B-CAN_N: track 78.1 -> 0.00 mm, vias 1 -> 0
- net /CAN_CS_B: track 59.3 -> 0.00 mm, vias 1 -> 0
- net /SCK: track 70.0 -> 28.1 mm
- net /CAN_INT: track 111.5 -> 69.7 mm
- net /MOSI: track 84.8 -> 43.0 mm
- net /MISO: track 77.5 -> 35.7 mm
- net +5V: track 106.9 -> 79.5 mm
- net Net-(Q3-G): track 25.5 -> 31.4 mm, vias 2 -> 1
- net Net-(Q2-G): track 29.7 -> 35.6 mm, vias 2 -> 1
- net Net-(J2-Pin_2): track 18.3 -> 23.4 mm
- net Net-(J2-Pin_3): track 15.1 -> 20.1 mm
- net /C-CAN_P: track 72.0 -> 71.2 mm, vias 1 -> 3
- net /C-CAN_N: track 72.5 -> 72.1 mm, vias 1 -> 3
Other:
- board text added: "Soul PS Dash V1.0"
- board text added: "github.com/eymenyg/hyundai_dash_v1"
- board text removed: "Hyundai Dash V1"

Commit message: KiCad: Soul.pcb: re-add IC markings on silkscreen
Other:
- board text added: "Soul PS Dash V1.1"
- board text removed: "Soul PS Dash V1.0"
Changed lines of the file:
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@@
 		)
 		(property "Value" "ULN2803A"
-			(at 3.81 22.65 0)
-			(layer "F.Fab")
+			(at 3.805 10.16 270)
+			(unlocked yes)
+			(layer "F.SilkS")
 			(effects
 				(font
@@
 		)
 		(property "Value" "ULN2803A"
-			(at 3.81 22.65 90)
-			(layer "F.Fab")
+			(at 3.805 10.16 180)
+			(layer "F.SilkS")
 			(effects
 				(font
@@
 		)
 		(property "Value" "74HC595"
-			(at 3.81 20.11 180)
-			(layer "F.Fab")
+			(at 3.805 8.89 270)
+			(layer "F.SilkS")
 			(effects
 				(font
@@
 		)
 	)
-	(gr_text "Soul PS Dash V1.0"
+	(gr_text "Soul PS Dash V1.1"
 		(locked yes)
 		(at 175.25 98.25 0)
